Commit message: [truckasaurus] added URDF for the robot with all measurements

File: linorobot2_description/urdf/mech/wheel.urdf.xacro (robot description, xacro)
@@ -1,5 +1,5 @@
 <?xml version="1.0"?>
 <robot xmlns:xacro="http://ros.org/wiki/xacro">
-  <xacro:macro name="wheel" params="side radius width pos_x pos_y pos_z mass">
+  <xacro:macro name="wheel" params="side radius width pos_x pos_y pos_z mass parent_link">
     <link name="${side}_wheel_link">
       <visual>
@@ -17,4 +17,12 @@
           <cylinder radius="${radius}" length="${width}"/>
         </geometry>
+        <surface>
+          <friction>
+            <ode>
+              <mu>0.5</mu>
+              <mu2>1.0</mu2>
+            </ode>
+          </friction>
+        </surface>
       </collision>
       <inertial>
@@ -38,8 +46,10 @@
     <joint name="${side}_wheel_joint" type="continuous">
       <axis xyz="0 1 0" />
-      <parent link="base_link"/>
+      <parent link="${parent_link}"/>
       <child link="${side}_wheel_link"/>
       <origin xyz="${pos_x} ${pos_y} ${pos_z}" rpy="0 0 0"/>
     </joint>
+    <gazebo reference="${side}_wheel_joint">
+    </gazebo>
   </xacro:macro>
 </robot>
