Commit message: - Reduce ekf frequency to 10 - set wheel_max_steer to correct value - set Ackermann min (reverse) velocity to same magnitude as forward - navigation.yaml   - set use_sim_time to False everywhere   - bt_navigator     - increase loop duration to 50ms   - controller     - set robot parameters for Truckasaurus     - allow tighter obstacle dist, smaller inflation     - favor forward drive = 10.0   - global costmap & local costmap     - update freq 5.0     - use footprint of Truckasaurus     - reduce inflation radius

File: linorobot2_description/urdf/controllers/ackermann_drive.urdf.xacro (robot description, xacro)
@@ -15,5 +15,5 @@
         <wheel_radius>${wheel_radius}</wheel_radius>
         <!--max_wheel_acceleration>1.0</max_wheel_acceleration-->
-        <min_velocity>-1.0</min_velocity>
+        <min_velocity>-2.0</min_velocity>
         <max_velocity>2.0</max_velocity>
         <min_acceleration>-1.0</min_acceleration>

File: linorobot2_description/urdf/truckasaurus_properties.urdf.xacro (robot description, xacro)
@@ -13,5 +13,5 @@
   <xacro:property name="wheel_mass" value="0.113" />
   <xacro:property name="wheel_torque" value="20" />
-  <xacro:property name="wheel_max_steer" value="1.396" />
+  <xacro:property name="wheel_max_steer" value="0.698" />
   <xacro:property name="wheel_mass_steering" value=".1" />
   <xacro:property name="kingpin_width" value="0.131" />
