Commit message: Adjusted ekf odom0 and imu0 config, minor  params adjustments,  imu urdf origin, add patches for nav2 launch files to disable AMCL and remove spin behavior

File: linorobot2_description/urdf/robots/truckasaurus.urdf.xacro (robot description, xacro)
@@ -81,7 +81,7 @@
     <xacro:insert_block name="laser_pose" />
   </xacro:generic_laser>
-  <xacro:depth_sensor>
+  <!-- <xacro:depth_sensor>
     <xacro:insert_block name="depth_sensor_pose" />
-  </xacro:depth_sensor>
+  </xacro:depth_sensor> -->
   <xacro:depthai_camera
    camera_name = "${depth_camera_name}"

File: linorobot2_description/urdf/sensors/generic_laser.urdf.xacro (robot description, xacro)
@@ -9,5 +9,5 @@
       max_angle="3.1416"
       min_range="0.08"
-      max_range="12.0"
+      max_range="17.0"
       frame_id="laser"
       topic_name="scan"

File: linorobot2_description/urdf/sensors/imu.urdf.xacro (robot description, xacro)
@@ -5,5 +5,5 @@
       <parent link="base_link"/>
       <child link="imu_link"/>
-      <origin xyz="0 0 0" rpy="0 0 0"/>
+      <origin xyz="0.085 -0.07 0.0" rpy="0 0 0"/>
     </joint>
     <gazebo reference="imu_link">

Commit message: Added GPS support - to URDF files - to bringup - to ekf with dual ekf and navsat_transform

File: linorobot2_description/urdf/robots/truckasaurus.urdf.xacro (robot description, xacro)
@@ -10,4 +10,5 @@
   <xacro:include filename="$(find linorobot2_description)/urdf/sensors/oakd_on_ptbase.urdf.xacro" />
   <xacro:include filename="$(find linorobot2_description)/urdf/controllers/ackermann_drive.urdf.xacro" />
+  <xacro:include filename="$(find linorobot2_description)/urdf/sensors/ultimate_gps.urdf.xacro" />
   <!--xacro:include filename="$(find linorobot2_description)/urdf/sensors/depth_sensor.urdf.xacro" /-->
   <xacro:base
@@ -78,4 +79,7 @@
   />
   <xacro:imu/>
+  <xacro:ultimate_gps>
+    <xacro:insert_block name="gps_sensor_pose" />
+  </xacro:ultimate_gps>
   <xacro:generic_laser>
     <xacro:insert_block name="laser_pose" />

File: linorobot2_description/urdf/truckasaurus_properties.urdf.xacro (robot description, xacro)
@@ -23,4 +23,7 @@
     <origin xyz="0.191 0 0.110" rpy="0 0 0"/>
   </xacro:property>
+  <xacro:property name="gps_sensor_pose">
+      <origin xyz="-0.235 0.0 0.055" rpy="0 0 0"/>
+  </xacro:property>
   <!-- OakD as depth sensor -->
   <xacro:property name="depth_camera_name" value="oak" />
