Commit message: [Truckasaurus] Worked on ekf_gps settings a lot - added Madgwick filter to bring up and config file for it - added fake_gps publisher script - changed location of IMU in urdf

File: linorobot2_description/urdf/sensors/imu.urdf.xacro (robot description, xacro)
@@ -5,5 +5,5 @@
       <parent link="base_link"/>
       <child link="imu_link"/>
-      <origin xyz="0.085 -0.07 0.0" rpy="0 0 0"/>
+      <origin xyz="-0.191 -0.075 0.016" rpy="0 0 0"/>
     </joint>
     <gazebo reference="imu_link">
@@ -24,5 +24,5 @@
           <xyzOffset>0 0 0</xyzOffset>
           <rpyOffset>0 0 0</rpyOffset>
-          <frameName>imu_link</frameName>
+          <frameName>imu_link_ned</frameName>
           <initialOrientationAsReference>false</initialOrientationAsReference>
       </plugin>
